Commit message: Imported upstream version '1.4.1' of 'upstream'

File: config/srdf/disable_collisions/tiago_pro_no-arm-left.srdf.xacro (robot description, xacro)
@@ -144,4 +144,6 @@
     <disable_collisions link1="arm_right_7_link" link2="torso_head_link" reason="Never"/>
     <disable_collisions link1="arm_right_7_link" link2="virtual_base_laser_link" reason="Never"/>
+    <disable_collisions link1="arm_right_7_link" link2="gripper_right_camera_link" reason="Never"/>
+    <disable_collisions link1="arm_right_tool_link" link2="gripper_right_camera_link" reason="Never"/>
     <disable_collisions link1="arm_right_tool_link" link2="base_footprint" reason="Never"/>
     <disable_collisions link1="arm_right_tool_link" link2="base_imu_link" reason="Never"/>

File: config/srdf/disable_collisions/tiago_pro_no-arm-right.srdf.xacro (robot description, xacro)
@@ -144,4 +144,6 @@
     <disable_collisions link1="arm_left_7_link" link2="torso_head_link" reason="Never"/>
     <disable_collisions link1="arm_left_7_link" link2="virtual_base_laser_link" reason="Never"/>
+    <disable_collisions link1="arm_left_7_link" link2="gripper_left_camera_link" reason="Never"/>
+    <disable_collisions link1="arm_left_tool_link" link2="gripper_left_camera_link" reason="Never"/>
     <disable_collisions link1="arm_left_tool_link" link2="base_footprint" reason="Never"/>
     <disable_collisions link1="arm_left_tool_link" link2="base_imu_link" reason="Never"/>

File: config/srdf/tiago_pro.srdf.xacro (robot description, xacro)
@@ -10,4 +10,5 @@
     <xacro:arg name="end_effector_left" default="pal-hey5"/>
     <xacro:arg name="end_effector_right" default="pal-hey5"/>
+    <xacro:arg name="has_teleop_arms" default="False"/>
     <xacro:arg name="ft_sensor_left" default="rokubi"/>
     <xacro:arg name="ft_sensor_right" default="rokubi"/>
@@ -20,4 +21,5 @@
     <xacro:property name="end_effector_right" value="$(arg end_effector_right)"/>
     <xacro:property name="end_effector_right_arg" value="$(arg end_effector_right)"/>
+    <xacro:property name="has_teleop_arms" value="$(arg has_teleop_arms)"/>
     <xacro:property name="ft_sensor_left" value="$(arg ft_sensor_left)"/>
     <xacro:property name="ft_sensor_right" value="$(arg ft_sensor_right)"/>
@@ -52,4 +54,14 @@
             <group name="torso" />
         </group>
+        <group name="arm_teleop_${side}">
+            <joint name="arm_teleop_${side}_1_joint" />
+            <joint name="arm_teleop_${side}_2_joint" />
+            <joint name="arm_teleop_${side}_3_joint" />
+            <joint name="arm_teleop_${side}_4_joint" />
+            <joint name="arm_teleop_${side}_5_joint" />
+            <joint name="arm_teleop_${side}_6_joint" />
+            <joint name="arm_teleop_${side}_7_joint" />
+            <!-- <joint name="arm_teleop_${side}_tool_joint" /> -->
+        </group>
     </xacro:macro>
     <xacro:if value="${has_arm_left}">
@@ -64,4 +76,11 @@
             <group name="arm_right" />
             <group name="arm_left" />
+        </group>
+    </xacro:if>
+    <!-- if has_teleop create a group arm with arm_teleop_left and arm_teleop right -->
+    <xacro:if value="${has_teleop_arms}">
+        <group name="arms_teleop">
+            <group name="arm_teleop_left" />
+            <group name="arm_teleop_right" />
         </group>
     </xacro:if>
@@ -97,4 +116,7 @@
         <xacro:property name="config_right" value="no-arm-right"/>
     </xacro:unless>
+    <xacro:if value="${has_teleop_arms}">
+        <xacro:include filename="$(find tiago_pro_moveit_config)/config/srdf/teleop_arms.srdf.xacro"/>
+    </xacro:if>
     <xacro:include filename="$(find tiago_pro_moveit_config)/config/srdf/disable_collisions/${robot}_${config_left}_${config_right}.srdf.xacro" />
 </robot>
